Commit message: changed scout_ros2 remote to fork

File: scout_description/urdf/scout_mini/scout_mini.urdf (robot description, URDF)
Before this commit: robot scout_mini, 7 links, 6 joints
Links:
- link base_link: geometry collision box size=0.595 0.395 0.13; visual mesh filename=package://scout_description/meshes/scout_mini/mini_base_lin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
- link front_left_wheel_link: geometry collision cylinder length=0.0852 radius=0.0875; visual mesh filename=package://scout_description/meshes/scout_mini/mini_wheel.dae
- link front_right_wheel_link: geometry collision cylinder length=0.0852 radius=0.0875; visual mesh filename=package://scout_description/meshes/scout_mini/mini_wheel.dae
- link rear_left_wheel_link: geometry collision cylinder length=0.0852 radius=0.0875; visual mesh filename=package://scout_description/meshes/scout_mini/mini_wheel.dae
- link rear_right_wheel_link: geometry collision cylinder length=0.0852 radius=0.0875; visual mesh filename=package://scout_description/meshes/scout_mini/mini_wheel.dae

File: scout_description/urdf/scout_mini/scout_mini.xacro (robot description, xacro)
@@ -21,5 +21,5 @@
             <origin xyz="0 0 0" rpy="0 0 0" />
             <geometry>
-                <mesh filename="package://scout_description/meshes/scout_mini/mini_base_link.dae" />
+                <mesh filename="package://scout_description/meshes/scout_mini/scout_mini/mini_base_link.dae" />
             </geometry>
         </visual>
